File: LCmeter0-LCD-8pinlcd-PIC_COMP.brd (EAGLE design)
At the start: 34 parts, among them IC1 PIC16F876A-X/SP-COMP-B-A/V, J1 HD44780, J2 PIC-UART, J3 PIC-ICSPICSP, K2 DS2Y, Q1 20MHz, T1 BC547, X1 FREQ, X2 L/C

Commit message: ...
Parts:
- JP1: value (none) -> CONN-2P2P/V; device pinhead:1X02 -> pinconn:CONN-2P-V
- moved JP1 1.80 mm to (53.3, 1.27), turned to 0 degrees
Connections:
- net GND: now also JP1.1; no longer JP1.2
- net VCC: now also JP1.2; no longer JP1.1
Routing:
- net GND: track 190.5 -> 175.3 mm
- net FREQ: track 38.1 -> 40.6 mm

Commit message: ...
Parts:
- L1: value 100μH -> 100µH; device r:L-02/5 -> l:L-02/5V
- S1: value SL-SW-2P-2T -> SW-2P-2T
- moved S1 7.62 mm to (3.81, 40.6), turned to 90 degrees
- moved L1 2.54 mm to (12.7, 43.2)
- moved J2 1.80 mm to (53.3, 12.7), turned to 0 degrees
- turned Q1 to 180 degrees
- renumbered U$1 to S2
Routing:
- net N$7: track 16.3 -> 27.9 mm, vias 0 -> 2
- net GND: track 175.3 -> 185.4 mm
- net /LC: track 73.5 -> 81.1 mm, vias 2 -> 4
- net M-: track 20.3 -> 27.9 mm, vias 2 -> 0
- net M+: track 20.3 -> 27.9 mm
- net N$2: track 35.6 -> 30.5 mm
