File: Headphone-Amplifier-ClassAB-alt2.brd (EAGLE design)
At the start: 40.6 x 17.8 mm, 17 parts, among them T1 2N3904, T2 2N3904, T3 2N3906

Commit message: ...
Parts:
- moved C3 1.80 mm to (29.2, 3.81)
- moved C1 1.27 mm to (8.89, 15.2)
- moved C2 1.27 mm to (8.89, 10.2)
- moved BAT 1.27 mm to (38.1, 3.81)
- moved IN 1.27 mm to (2.54, 3.81)
- moved HDPH 1.27 mm to (38.1, 14.0)
Changed lines of the file:
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@@
       </autorouter>
       <elements>
-        <element name="BAT" library="pad" package="SPAD+-" value="SPAD+-+-" x="38.1" y="5.08" />
-        <element name="C1" library="c" package="E2,5-3" value="4.7uF" x="7.62" y="15.24" rot="R180" />
-        <element name="C2" library="c" package="E2,5-3" value="4.7uF" x="7.62" y="10.16" rot="R180" />
-        <element name="C3" library="c" package="E5-5" value="470uF" x="30.48" y="2.54" rot="R270" />
+        <element name="BAT" library="pad" package="SPAD+-" value="SPAD+-+-" x="38.1" y="3.81" />
+        <element name="C1" library="c" package="E2,5-3" value="4.7uF" x="8.89" y="15.24" rot="R180" />
+        <element name="C2" library="c" package="E2,5-3" value="4.7uF" x="8.89" y="10.16" rot="R180" />
+        <element name="C3" library="c" package="E5-5" value="470uF" x="29.21" y="3.81" rot="R270" />
         <element name="C4" library="c" package="E2,5-5" value="100uF" x="25.4" y="7.62" />
         <element name="D1" library="d" package="DO34-5-V" value="1N4148" x="15.24" y="12.7" />
         <element name="D2" library="d" package="DO34-5V" value="1N4148" x="12.7" y="12.7" />
-        <element name="HDPH" library="pad" package="SPAD-+" value="SPAD+--+" x="38.1" y="15.24" />
-        <element name="IN" library="pad" package="SPAD-+" value="SPAD+--+" x="2.54" y="2.54" />
+        <element name="HDPH" library="pad" package="SPAD-+" value="SPAD+--+" x="38.1" y="13.97" />
+        <element name="IN" library="pad" package="SPAD-+" value="SPAD+--+" x="2.54" y="3.81" />
         <element name="R1" library="r" package="0204/10" value="100k" x="12.7" y="7.62" />
         <element name="R2" library="r" package="0204/10" value="330" x="25.4" y="12.7" />
