File: Headphone-Amplifier-ClassAB-alt4.sch (EAGLE design)
At the start: 17 parts, among them T1 BC547, T2 BC327, T3 BC337

Commit message: ...
Parts:
- T1: device t:BC547CBE -> t:BC547
Changed lines of the file:
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@@
 <?xml version="1.0" encoding="utf-8"?>
-<eagle version="7.6.0">
+<eagle version="7.2.0">
   <drawing>
     <settings>
@@
       <setting verticaltext="up" />
     </settings>
-    <grid distance="0.05" unitdist="inch" unit="inch" style="lines" multiple="2" display="yes" altdistance="0.025" altunitdist="inch" altunit="inch" />
+    <grid distance="0.1" unitdist="inch" unit="inch" style="lines" multiple="1" display="yes" altdistance="2" altunitdist="inch" altunit="inch" />
     <layers>
       <layer number="1" name="Top" color="4" fill="1" visible="no" active="no" />
@@
       <layer number="250" name="trash" color="7" fill="1" visible="yes" active="yes" />
     </layers>
-    <schematic xreflabel="%F%N/%S.%C%R" xrefpart="/%S.%C%R">
+    <schematic xreflabel="%F%N/%S" xrefpart="/%S.%C%R">
       <description>4x4 - Three Transistor Headphone Amplifier - Class AB
 http://www.electronics-diy.com/4x4.php</description>
@@
       </classes>
       <parts>
-        <part name="T1" library="t" deviceset="BC547" device="CBE" value="BC547" />
+        <part name="T1" library="t" deviceset="BC547" device="" value="BC547" />
         <part name="T2" library="t" deviceset="BC327" device="" value="BC327" />
         <part name="D1" library="d" deviceset="1N4148" device="34-5V" value="" />
