File: Headphone-Amplifier-ClassAB-alt.brd (EAGLE design)
At the start: 17 parts, among them T1 BC547, T2 2N3904, T3 2N3906

Commit message: ...
Parts:
- moved C1 1.27 mm to (8.89, 15.2)
- moved C2 1.27 mm to (8.89, 10.2)
- moved C3 1.27 mm to (27.9, 3.81)
- moved IN 1.27 mm to (2.54, 3.81)
- moved HDPH 1.27 mm to (38.1, 14.0)
Changed lines of the file:
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@@
       <elements>
         <element name="BAT" library="pad" package="SPAD+-" value="SPAD+-+-" x="35.56" y="2.54" rot="R270" />
-        <element name="C1" library="c" package="E2,5-4" value="4.7uF" x="7.62" y="15.24" rot="R180" />
-        <element name="C2" library="c" package="E2,5-4" value="4.7uF" x="7.62" y="10.16" rot="R180" />
-        <element name="C3" library="c" package="E5-5/V" value="100-1000uF" x="27.94" y="2.54" rot="R270" />
+        <element name="C1" library="c" package="E2,5-4" value="4.7uF" x="8.89" y="15.24" rot="R180" />
+        <element name="C2" library="c" package="E2,5-4" value="4.7uF" x="8.89" y="10.16" rot="R180" />
+        <element name="C3" library="c" package="E5-5/V" value="100-1000uF" x="27.94" y="3.81" rot="R270" />
         <element name="C4" library="c" package="E5-4" value="220uF" x="25.4" y="7.62" rot="R180" />
         <element name="D1" library="d" package="DO34-5V" value="1N4148" x="15.24" y="12.7" />
         <element name="D2" library="d" package="DO34-5V" value="1N4148" x="12.7" y="12.7" />
-        <element name="HDPH" library="pad" package="SPAD+-" value="SPAD+-+-" x="38.1" y="15.24" rot="R180" />
-        <element name="IN" library="pad" package="SPAD+-" value="SPAD+-+-" x="2.54" y="2.54" />
+        <element name="HDPH" library="pad" package="SPAD+-" value="SPAD+-+-" x="38.1" y="13.97" rot="R180" />
+        <element name="IN" library="pad" package="SPAD+-" value="SPAD+-+-" x="2.54" y="3.81" />
         <element name="R1" library="r" package="0204/7" value="100k" x="12.7" y="7.62" />
         <element name="R2" library="r" package="0204/7" value="330" x="25.4" y="12.7" />

Commit message: ...
Parts:
- C1, C2: device c:E2,5-4 -> c:E2,5-3
- C3: device c:E5-5/V -> c:E2.5-4/V
- D1: device d:DO34-5V -> d:DO34-5-V
- HDPH: value SPAD+-+- -> SPAD+--+; device pad:SPAD+- -> pad:SPAD-+
- R1, R2, R3, R4: device r:0204/7 -> r:0204/10
- R5: device r:POT -> r:CONN-3P
- moved BAT 2.84 mm to (38.1, 3.81), turned to 0 degrees
- moved R2 2.54 mm to (27.9, 12.7)
- moved R3 2.54 mm to (27.9, 15.2)
- moved C3 2.54 mm to (30.5, 3.81), turned to 0 degrees
- turned IN to 180 degrees
- turned R5 to 180 degrees
Connections:
- net GND: now also R5.3; no longer R5.E
- net N$5: now also R5.1; no longer R5.A
- net N$6: now also R5.2; no longer R5.S
Routing:
- net GND: track 0.00 -> 43.2 mm
- net N$8: track 0.00 -> 38.1 mm
- net N$9: track 0.00 -> 17.8 mm
- net N$10: track 0.00 -> 15.2 mm
- net N$2: track 0.00 -> 12.7 mm
- net N$1: track 0.00 -> 10.2 mm
- net N$5: track 0.00 -> 7.62 mm
- net N$7: track 0.00 -> 7.62 mm
- net T3: track 0.00 -> 7.62 mm
- net V+: track 0.00 -> 5.08 mm
- net N$3: track 0.00 -> 2.54 mm
- net N$6: track 0.00 -> 2.54 mm
Other:
- board outline added: 40.6 x 17.8 mm
