File: Headphone-Amplifier-ClassAB-alt.sch (EAGLE design)
At the start: 17 parts, among them T1 BC547, T2 2N3904, T3 2N3906

Commit message: ...
Parts:
- C1, C2: device c:CPOLE2,5-4 -> c:CPOLE2,5-3
- C3: device c:CPOLE5-5/V -> c:CPOLE2,5-4/V
- D1: device d:1N414834-5V -> d:DIODE34-5-V
- D2: device d:1N414834-5V -> d:DIODE34-5V
- HDPH: value SPAD+-+- -> SPAD+--+; device pad:SPAD+-+- -> pad:SPAD+--+
- R1, R2, R4: device r:R-H0204/7 -> r:R-H0204/10
- R3: device r:R0204/7 -> r:R0204/10
- R5: device r:POT -> r:POT-3P
